Commit message: debugging

File: assets/urdf/cartpole.urdf (robot description, URDF)
Before this commit: robot physics, 4 links, 3 joints
Links:
- added link ground_plane, mass 0; collision box size=30 30 0.1; visual box size=30 30 0.1
Joints:
- added joint ground_joint: type fixed, parent world, child ground_plane, origin xyz=0 0 0
- joint cart_to_pole: origin xyz=0.0 0.0 0 -> (none)
- joint slider_to_cart: origin xyz=0.0 0.0 0.0 -> (none)
